File: KiCAD/LibreDAB/LibreDAB.kicad_sch (KiCad schematic)
At the start: 15 parts

Commit message: Initial kicad schematic draft
Other:
- company: (none) -> Fairflow Energy
- title: Micro-inverter - 450W -> LibreDAB - 800 W
