File: KiCAD/LibreDAB/Microcontroller.kicad_sch (KiCad schematic)
At the start: 22 parts, among them U901 OwnTech_SPIN, U902 WE-TVS-824015043, U903 WE-TVS-824015043

Commit message: Initial kicad schematic draft
Parts:
- U901: footprint Footprints:OwnTech_SPINTHT_1 -> project:OwnTech_SPINTHT_1
Changed lines of the file:
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@@
 			)
 		)
-		(property "Footprint" "Footprints:OwnTech_SPINTHT_1"
+		(property "Footprint" "project:OwnTech_SPINTHT_1"
 			(at 114.3 93.98 0)
 			(effects
@@
 			)
 		)
-		(property "Footprint" "Footprints:OwnTech_SPINTHT_1"
+		(property "Footprint" "project:OwnTech_SPINTHT_1"
 			(at 40.64 113.03 0)
 			(effects
@@
 			)
 		)
-		(property "Footprint" "Footprints:OwnTech_SPINTHT_1"
+		(property "Footprint" "project:OwnTech_SPINTHT_1"
 			(at 53.34 30.48 0)
 			(effects
@@
 			)
 		)
-		(property "Footprint" "Footprints:OwnTech_SPINTHT_1"
+		(property "Footprint" "project:OwnTech_SPINTHT_1"
 			(at 39.37 91.44 0)
 			(effects
