File: KiCAD/LibreDAB/current.kicad_sch (KiCad schematic)
At the start: 22 parts, among them U201 MCP6486UT-E/LT, U5 AMC1301DWR, U8 MCP6486UT-E/LT

Commit message: Schematic updates still setting up
Parts:
- renumbered C202 to C10, C203 to C11, C46 to C12, C47 to C13, C42 to C14, C205 to C15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
