File: KiCAD/LibreDAB/power.kicad_sch (KiCad schematic)
At the start: 170 parts, among them J1 Conn_01x01, J2 Conn_01x01, J3 Conn_01x01, J5 Conn_01x01, J8 Conn_01x01, K1 HF140FF/012-2HSWTF, Q1 CID12N65D, Q10 CJAC90SN12, Q11 ZXMN7A11GTA, Q2 CID12N65D, Q3 CID12N65D, Q4 CID12N65D, Q5 CJAC90SN12, Q6 CJAC90SN12, Q7 CJAC90SN12, Q8 CJAC90SN12, Q9 CJAC90SN12, T1 Transformer_1P_1S, T2 Transformer_1P_1S, U1 INA240A1PWR, U2 INA240A1PWR, U3 UCC27282DRC, U4 UCC27282DRC

Commit message: Initial kicad schematic draft
Parts:
- removed C1, C12, C14, C3: 1uF, Capacitor_SMD:C_0805_2012Metric, symbol Device:C_Small
- removed C10, C116, C117, C5: 4.7nF, Capacitor_THT:C_Rect_L13.0mm_W6.0mm_P10.00mm_FKS3_FKP3_MKS4, symbol Device:C_Small
- removed C101, C102, C13, C15: 4.7uF, Capacitor_SMD:C_0805_2012Metric, symbol Device:C_Small
- removed C103, C104, C105, C106, C107, C108, C109, C110, C128, C129, C130, C131, C132, C133, C134, C135, C18, C19, C20, C21, C23, C24, C25, C26, C29, C30, C31, C32, C34, C35, C36, C37: 4.7uF, Footprints:C_1210_3225Metric, symbol Device:C
- removed C11, C54: 2.2nF, Capacitor_THT:C_Rect_L9.0mm_W4.0mm_P7.50mm_MKT, symbol Device:C_Small
- removed C111: 47uF, Capacitor_SMD:C_Elec_10x10.2, symbol Device:C_Polarized
- removed C113, C122: 120nF, Capacitor_THT:C_Rect_L13.0mm_W6.0mm_P10.00mm_FKS3_FKP3_MKS4, symbol Device:C_Small
- removed C114, C115, C16, C17: 100nF, Capacitor_SMD:C_1210_3225Metric, symbol Device:C
- removed C118, C119: 1nF, Footprints:C_TH_L6.3-W4.4-P10.00-D0.6-S3.8, symbol Device:C_Small
- removed C120, C125, C126: 1nF, Capacitor_THT:C_Rect_L10.3mm_W4.5mm_P7.50mm_MKS4, symbol Device:C_Small
- removed C123, C124: 2.2nF, Capacitor_THT:C_Rect_L10.3mm_W4.5mm_P7.50mm_MKS4, symbol Device:C_Small
- removed C127: 1uF, Capacitor_THT:C_Rect_L18.0mm_W8.0mm_P15.00mm_FKS3_FKP3, symbol Device:C_Small
- removed C136, C137: 1nF, Capacitor_SMD:C_0603_1608Metric, symbol Device:C_Small
- removed C22, C27, C33, C38: 1uF, Capacitor_THT:C_Rect_L18.0mm_W8.0mm_P15.00mm_FKS3_FKP3, symbol Device:C
- removed C39: 100nF, Capacitor_SMD:C_0805_2012Metric, symbol Device:C_Small
- removed C40, C53, C8, C9: 470nF, Capacitor_SMD:C_0603_1608Metric, symbol Device:C_Small
- removed C6: 120µF, Footprints:C_film_capacitors_board, symbol Device:C
- removed C7: 680nF, Capacitor_THT:C_Rect_L18.0mm_W9.0mm_P15.00mm_FKS3_FKP3, symbol Device:C_Small
- removed D1, D2, D3, D4: D_Schottky, Footprints:TO-252-2_Diode, symbol Device:D_Schottky
- removed D101, D102: ES1JW, Footprints:D_SOD-123, symbol Device:D
- removed D5: 40V - BAT165E6327F, Diode_SMD:D_SOD-323, symbol Device:D_Schottky
- removed F1, F101: 2.5A, Footprints:FUSE-TH_L8.4-W4.1-P5.08-D0.6, symbol Device:Fuse
- removed FB1, FB2: 300@100MHz, Inductor_SMD:L_1206_3216Metric, symbol Device:FerriteBead_Small
- removed FL1, FL2: 5mH, Footprints:Choke_TH_XRSQ1515-5MH-V-1013, symbol Device:L_Coupled_1243
- removed FL3: 1mH, Footprints:Choke_TH_4P-L23.0-W15.0-P7.50-D1.0-S9.0, symbol Device:L_Coupled_1243
- removed GD1: 2R600B-8S, Footprints:SMD_GDT, symbol Device:GDT_2Pin
- removed HS101, HS104, HS105, HS106, HS107, HS108, HS109, HS11, HS110, HS111, HS12, HS5: 5x3mm pad 3mm high, Footprints:Heatsink_BTC-533-ZN01, symbol Mechanical:Heatsink_Pad
- removed J1, J2, J3, J5, J8: Conn_01x01, Footprints:Connector_SMD-4_TS34056055-0440, symbol Symbols:Conn_01x01
- removed K1: HF140FF/012-2HSWTF, Footprints:RELAY-TH_HF140FF-024-2HSWT, symbol Symbols:HF140FF/012-2HSWTF
- removed L1, L3: 250uH, Footprints:L_SMD_L28.0-W23-LS25, symbol Device:L
- removed L6: 33uH, Footprints:L_SRP1510CA-330M, symbol Device:L
- removed Logo101: ~, Footprints:owntech21mm, symbol Symbols:Logo
- removed Q10, Q5, Q6, Q7, Q8, Q9: CJAC90SN12, Footprints:DFN-8-1EP_5x6_P1.27mm, symbol Transistor_FET:Q_NMOS_SGD
- removed Q11: ZXMN7A11GTA, Package_TO_SOT_SMD:SOT-223, symbol Transistor_FET:Q_NMOS_GDSD
- removed R1, R2, R4, R5: 33, Resistor_SMD:R_0805_2012Metric, symbol Device:R_Small
- removed R10: 5mR, Resistor_SMD:R_2512_6332Metric, symbol Device:R_Small
- removed R101, R109, R32, R33, R8: 20k, Resistor_SMD:R_0603_1608Metric, symbol Device:R_Small
- removed R102, R103: 3.3R, Resistor_SMD:R_0805_2012Metric, symbol Device:R_Small
- removed R104, R105, R106, R107, R108: 20, Resistor_SMD:R_0603_1608Metric, symbol Device:R_Small
- removed R110, R9: 10k, Resistor_SMD:R_0603_1608Metric, symbol Device:R_Small
- removed R12: 47R, Resistor_SMD:R_0805_2012Metric, symbol Device:R
- removed R13: 10k, Resistor_SMD:R_0805_2012Metric, symbol Device:R
- removed R3: 4.7R, Resistor_SMD:R_2512_6332Metric, symbol Device:R_Small
- removed RV1, RV2, RV3: 14D621, Footprints:RV_Disc_D15.5mm_W11mm_P7.5mm, symbol Device:Varistor
- removed RV101, RV102, RV103: TMOV14RP275, Varistor:RV_Disc_D12mm_W6.2mm_P7.5mm, symbol Device:Varistor
- removed T1, T2: Transformer_1P_1S, Footprints:RM12, symbol Symbols:Transformer_1P_1S
- removed TP101, TP103, TP105, TP107: TestPoint_Probe, Footprints:TestPoint_Pad_D0.5mm, symbol Connector:TestPoint_Probe
- removed TP102, TP104, TP106, TP108, TP109: TestPoint_Probe, Footprints:TestPoint_Pad_D1.0mm, symbol Connector:TestPoint_Probe
- removed U1, U2: INA240A1PWR, Package_SO:TSSOP-8_4.4x3mm_P0.65mm, symbol Amplifier_Current:INA240A1PW
- removed U3, U4: UCC27282DRC, Footprints:VSON-10_L3.0-W3.0-P0.50-TL-EP, symbol Symbols:UCC27282DRC
- added J1: Wago 4 contacts, Footprints:WAGO-2604-1104, symbol Symbols:Wago 4 contacts
- added TR1: TRANSF1, project:RM12, symbol Transformer:TRANSF1
- added U1, U2: LMG2100R026VBNR, VBN0018A-MFG:VBN0018A-MFG, symbol LMG2100R026VBNR:LMG2100R026VBNR
- added U4: INA240A1PWR, Package_SO:TSSOP-8_4.4x3mm_P0.65mm, symbol Amplifier_Current:INA240A1PW
- L5: footprint Footprints:L_SRP1510CA-330M -> project:L_SRP1510CA-330M
- Q1, Q2, Q3, Q4: value CID12N65D -> ~; footprint Footprints:DFN-10_L8.0-W6.0_CID12N65D -> project:DFN-10_L8.0-W6.0_CID12N65D; LCSC C21547657 -> (none); Rotation Offset 90 -> (none)
Connections:
- net +12V_{HV}: no longer names the net of Q4.6 (VCC)
- net +12V_{HV}: no longer Q3.6 (VCC)
- net +12V_{SN1}: no longer names the net of Q2.6 (VCC)
- net +12V_{SN2}: no longer names the net of Q1.6 (VCC)
- net +5V_{DGND}: no longer names the net of C28.1
- net +5V_{DGND}: now also U4.5 (V+)
- removed net GND_{HV}: C121.2, Q3.11 (PGND), Q3.12 (S), Q3.7 (SGND), Q4.11 (PGND), Q4.12 (S), Q4.7 (SGND)
- net GND_{LV}: no longer names the net of C112.2
- net GND_{LV}: no longer C28.2
- net HV_{BUS} renamed DC Voltage sense/In+
- net DC Voltage sense/In+: now also Q3.1 (D), J1.1 (Pin_1); no longer Q2.1 (D)
- net LSW1: no longer names the net of L5.2
- net LSW1: now also U1.7 (VIN), U2.7 (VIN)
- net PWM_{IIHigh1}: no longer names the net of Q2.8 (PWM)
- net PWM_{IIHigh2}: no longer names the net of Q1.8 (PWM)
- net PWM_{IILow1}: no longer names the net of Q3.8 (PWM)
- net PWM_{IILow2}: no longer names the net of Q4.8 (PWM)
- removed net SN1: Q2.11 (PGND), Q2.12 (S), Q2.7 (SGND), Q3.1 (D)
- removed net SN2: Q1.11 (PGND), Q1.12 (S), Q1.7 (SGND), Q4.1 (D)
- net ThPad_{IND1}: no longer names the net of L5.1, R7.1
- net ThPad_{IND1}: now also U4.2 (+)
- net V_{ILow}: no longer names the net of C112.1
- net V_{ILow}: no longer R7.2
- new net: Q3.12 (S), Q4.1 (D)
- new net: TR1.1, U1.5 (SW)
- new net: Q1.12 (S), Q2.1 (D), TR1.3, TR1.4
- new net: TR1.2, U2.5 (SW)
- new net DC Voltage sense/In-: C121.2, J1.2 (Pin_2), Q2.12 (S), Q4.12 (S)
- new net Input voltage sense/In+: R7.2, U4.3 (-)
- new net Input voltage sense/In-: C28.2, U1.15 (AGND), U2.15 (AGND), U4.1 (GND), U4.4 (GND), U4.6 (REF2), U4.7 (REF1)
Other:
- removed sheet AC Current sense
- removed sheet Grid Voltage sense
- note removed: "0.6mA@12V"
- note removed: "2.5mA@5V"
- note removed: "67mA@12V"
- note removed: "A"
- note removed: "Current range: 0-8 A Max shunt drop: 40 mV @ 8 A INA240A1: gain = 20 V/V → VOUT ≈ 0.8 V @ 8 A Measurement resolution (12-bit ADC, 2.048 V): ≈ 5 mA / LSB"
- note removed: "Fast decoupling caps placed Close to half bridges"
- note removed: "INA240A1PWR REFs to GND for unidirectional measurements"
- note removed: "Low Side Drivers"
- note removed: "Low gate threshold to be driven directly by MCU"
- note removed: "P=I2R=64*0,005=0,32 W"
- note removed: "Relay for grid connection When PLL synched"
- note removed: "Surge protection"
- note removed: "Thermal connections to chassis. Plain copper standoffs"
- note removed: "V"
- moved on the sheet: C112, C121, C28, L5, R7

Commit message: Schematic updates still setting up
Parts:
- removed C112: 47uF, Capacitor_SMD:C_Elec_10x10.2, symbol Device:C_Polarized
- removed unit 2 of J1
- removed L5: 33uH, project:L_SRP1510CA-330M, symbol Device:L
- removed R7: 5mR, Resistor_SMD:R_2512_6332Metric, symbol Device:R_Small
- removed U4: INA240A1PWR, Package_SO:TSSOP-8_4.4x3mm_P0.65mm, symbol Amplifier_Current:INA240A1PW
- added C102, C30, C31, C34: 4.7uF, project:C_0805_2012Metric, symbol Device:C_Small
- added C27: 2.2uF, Capacitor_THT:C_Rect_L18.0mm_W8.0mm_P15.00mm_FKS3_FKP3, symbol Device:C_Small
- added C29, C32, C33: 1uF, project:C_0805_2012Metric, symbol Device:C_Small
- added D1, D102: ES1JW, project:D_SOD-123, symbol Device:D
- added J2: Wago 4 contacts, Footprints:WAGO-2604-1104, symbol Symbols:Wago 4 contacts
- added R103, R18: 3.3R, project:R_0805_2012Metric, symbol Device:R_Small
- added R17, R19, R20, R21: 33, project:R_0805_2012Metric, symbol Device:R_Small
- added RV101, RV8: TMOV14RP275, Varistor:RV_Disc_D12mm_W6.2mm_P7.5mm, symbol Device:Varistor
- C28: value 100nF -> 1uF; footprint Capacitor_SMD:C_0805_2012Metric -> project:C_0805_2012Metric; LCSC C49678 -> C28323
Connections:
- net DC Voltage sense/In+: now also RV101.1
- net Input voltage sense/In+: now also U1.7 (VIN), U2.7 (VIN), C27.1, J2.2 (Pin_2), RV8.1
- net at C28.1: now also Q3.5 (VDD)
- net at Q3.12 (S), Q4.1 (D): now also TR1.3
- net at Q4.10 (OUT-): now also R21.2
- net at Q4.11 (PGND): now also Q4.7 (SGND), C33.2, C34.2
- net at Q4.5 (VDD): now also C33.1
- net +12V_{HV}: now reaches Q4.6 (VCC)
- net +12V_{HV}: now also Q2.6 (VCC), C31.1, C34.1, D1.2 (A), D102.2 (A)
- net at Q4.9 (OUT+): now also R21.1
- net at Q1.10 (OUT-): now also R19.2
- net at Q1.12 (S), Q2.1 (D), TR1.4: no longer TR1.3
- net at Q1.5 (VDD): now also C29.1
- net at Q1.6 (VCC): now also C30.1, R18.1
- net at Q1.7 (SGND): now also C29.2, C30.2
- net at Q1.9 (OUT+): now also R19.1
- net at Q3.10 (OUT-): now also R17.2
- net at Q3.11 (PGND): now also C28.2, Q3.7 (SGND), C102.2
- net at Q3.6 (VCC): now also C102.1, R103.1
- net at Q3.9 (OUT+): now also R17.1
- net at Q2.10 (OUT-): now also R20.2
- net at Q2.11 (PGND): now also Q2.7 (SGND), C31.2, C32.2
- net at Q2.5 (VDD): now also C32.1
- net at Q2.9 (OUT+): now also R20.1
- net DC Voltage sense/In- renamed AC Current sense1/In-
- net AC Current sense1/In-: no longer J1.2 (Pin_2)
- net Input voltage sense/In- renamed AC Current sense/In+
- net AC Current sense/In+: now also C27.2; no longer C28.2
- new net: D1.1 (K), R18.2
- new net: D102.1 (K), R103.2
- new net AC Current sense/In-: J2.1 (Pin_1), RV8.2
- new net AC Current sense1/In+: J1.2 (Pin_2), RV101.2
Other:
- added sheet AC Current sense (current.kicad_sch)
- added sheet AC Current sense1 (current.kicad_sch)
- note added: "400 V DC bus"
- note added: "Battery"
- moved on the sheet: C121, J1A, Q1, Q2, Q3, Q4, TR1, U1, U2
