File: KiCAD/LibreDAB/LV_Bridge.kicad_sch (KiCad schematic)
At the start: 66 parts, among them J1 HX PM2.54-1X4P TP H8.5-ZQ, J2 TS30050050-040, J3 TS30050050-040, J4 HX PM2.54-1X4P TP H8.5-ZQ, J5 HX PM2.54-1X4P TP H8.5-ZQ, J6 HX PM2.54-1X4P TP H8.5-ZQ, J7 TS30050050-040, J8 TS30050050-040, Q1 SP010N01BGHTO, Q2 SP010N01BGHTO, Q3 SP010N01BGHTO, Q4 SP010N01BGHTO, U2 10 MHz Opamp, U3 10 MHz Opamp, U4 10 MHz Opamp

Commit message: Initial routing complete
Connections:
- net GND: no longer R6.1
- net V_LV-: no longer R7.1
- new net GND_sense: R5.4 (Vsense2), R6.1
- new net V_LV-_sense: R5.3 (Vsense1), R7.1
Changed lines of the file:
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@@
 	(text "Ipeak = 60 A, bidirectional in short circuit condition\nSmallest 2512 Resistor is 0.5 mOhm\nCheck losses:\nI^2R = 60^2 * 0.5m = 1.8 Watts at short circuit condition\nI^2R = 35^2 * 0.5m = 0.61 Watts at max normal current\n\nCheck voltage drop:\nV = IR = 60*0.5m = 30 mV"
 		(exclude_from_sim no)
-		(at 79.248 110.998 0)
+		(at 79.248 116.078 0)
 		(effects
 			(font
@@
 	(wire
 		(pts
+			(xy 128.27 153.67) (xy 138.43 153.67)
+		)
+		(stroke
+			(width 0)
+			(type default)
+		)
+	)
+	(wire
+		(pts
 			(xy 220.98 135.89) (xy 226.06 135.89)
 		)
@@
 	(wire
 		(pts
+			(xy 87.63 96.52) (xy 87.63 102.87)
+		)
+		(stroke
+			(width 0)
+			(type default)
+		)
+	)
+	(wire
+		(pts
 			(xy 151.13 76.2) (xy 158.75 76.2)
 		)
@@
 	(wire
 		(pts
-			(xy 71.12 63.5) (xy 82.55 63.5)
+			(xy 95.25 96.52) (xy 95.25 100.33)
 		)
 		(stroke
@@
 	(wire
 		(pts
-			(xy 213.36 88.9) (xy 212.09 88.9)
+			(xy 71.12 63.5) (xy 82.55 63.5)
 		)
 		(stroke
@@
 	(wire
 		(pts
-			(xy 212.09 39.37) (xy 229.87 39.37)
+			(xy 213.36 88.9) (xy 212.09 88.9)
 		)
 		(stroke
@@
 	(wire
 		(pts
-			(xy 223.52 29.21) (xy 226.06 29.21)
+			(xy 212.09 39.37) (xy 229.87 39.37)
 		)
 		(stroke
@@
 	(wire
 		(pts
-			(xy 49.53 93.98) (xy 57.15 93.98)
+			(xy 223.52 29.21) (xy 226.06 29.21)
 		)
 		(stroke
@@
 	(wire
 		(pts
-			(xy 226.06 30.48) (xy 229.87 30.48)
+			(xy 49.53 93.98) (xy 57.15 93.98)
 		)
 		(stroke
@@
 	(wire
 		(pts
-			(xy 130.81 153.67) (xy 138.43 153.67)
+			(xy 226.06 30.48) (xy 229.87 30.48)
 		)
 		(stroke
@@
 	(wire
 		(pts
-			(xy 130.81 133.35) (xy 138.43 133.35)
+			(xy 128.27 133.35) (xy 138.43 133.35)
 		)
 		(stroke
@@
 		)
 	)
+	(label "GND_sense"
+		(at 95.25 100.33 0)
+		(effects
+			(font
+				(size 1.27 1.27)
+			)
+			(justify left bottom)
+		)
+	)
 	(label "LSW1"
 		(at 142.24 76.2 0)
@@
 		)
 	)
+	(label "V_LV-_sense"
+		(at 87.63 102.87 0)
+		(effects
+			(font
+				(size 1.27 1.27)
+			)
+			(justify left bottom)
+		)
+	)
 	(label "I_LVsense"
 		(at 226.06 135.89 0)
@@
 		)
 	)
+	(label "V_LV-_sense"
+		(at 128.27 153.67 0)
+		(effects
+			(font
+				(size 1.27 1.27)
+			)
+			(justify left bottom)
+		)
+	)
 	(label "PWM-L1"
 		(at 53.34 22.86 0)
@@
 		)
 	)
-	(label "V_LV-"
-		(at 130.81 153.67 0)
+	(label "GND_sense"
+		(at 128.27 133.35 0)
 		(effects
 			(font
@@
 		(pin "1"
 		)
+		(pin "4"
+		)
+		(pin "3"
+		)
 		(instances
 			(project ""
@@
 					(unit 1)
 				)
-			)
-		)
-	)
-	(symbol
-		(lib_id "power:GND")
-		(at 130.81 133.35 0)
-		(unit 1)
-		(exclude_from_sim no)
-		(in_bom yes)
-		(on_board yes)
-		(dnp no)
-		(fields_autoplaced yes)
-		(property "Reference" "#PWR018"
-			(at 130.81 139.7 0)
-			(effects
-				(font
-					(size 1.27 1.27)
-				)
-				(hide yes)
-			)
-		)
-		(property "Value" "GND"
-			(at 130.81 138.43 0)
-			(effects
-				(font
-					(size 1.27 1.27)
-				)
-			)
-		)
-		(property "Footprint" ""
-			(at 130.81 133.35 0)
-			(effects
-				(font
-					(size 1.27 1.27)
-				)
-				(hide yes)
-			)
-		)
-		(property "Datasheet" ""
-			(at 130.81 133.35 0)
-			(effects
-				(font
-					(size 1.27 1.27)
-				)
-				(hide yes)
-			)
-		)
-		(property "Description" "Power symbol creates a global label with name \"GND\" , ground"
-			(at 130.81 133.35 0)
-			(effects
-				(font
-					(size 1.27 1.27)
-				)
-				(hide yes)
-			)
-		)
-		(pin "1"
-		)
-		(instances
-			(project "LibreDAB"
-				(path "/daf77073-b189-4351-8636-4e7a5198e1b7/f3c2518b-d41d-4c2c-ab2c-6739c5137e70"
-					(reference "#PWR018")
-					(unit 1)
-				)

Commit message: Resolved various DRC issues. Almost ready for review
Parts:
- added D1: TVS DIODE 60VWM 96.8VC SMB(DO-214AA), lcsc_footprints:C49066953_SMB_L4_5-W3_7-LS5_4-RD, symbol lcsc_imported:SMBJ60A TVS
Connections:
- net V_LV+: now also D1.1 (K)
- net V_LV-: now also D1.2 (A)
Changed lines of the file:
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@@
 	(text "Stored energy: 0.5 CV^2\n0.5 * 45u * 80^2 = 0.144 J\nDischarge time constant: RC\n~ 1M * 47u = 45 seconds"
 		(exclude_from_sim no)
-		(at 38.862 79.756 0)
+		(at 29.972 79.502 0)
 		(effects
 			(font
@@
 	)
 	(junction
+		(at 49.53 63.5)
+		(diameter 0)
+		(color 0 0 0 0)
+	)
+	(junction
 		(at 128.27 22.86)
 		(diameter 0)
@@
 	)
 	(junction
+		(at 49.53 93.98)
+		(diameter 0)
+		(color 0 0 0 0)
+	)
+	(junction
 		(at 151.13 63.5)
 		(diameter 0)
@@
 	(wire
 		(pts
+			(xy 49.53 63.5) (xy 49.53 73.66)
+		)
+		(stroke
+			(width 0)
+			(type default)
+		)
+	)
+	(wire
+		(pts
 			(xy 50.8 170.18) (xy 55.88 170.18)
 		)
@@
 	(wire
 		(pts
+			(xy 49.53 83.82) (xy 49.53 93.98)
+		)
+		(stroke
+			(width 0)
+			(type default)
+		)
+	)
+	(wire
+		(pts
 			(xy 22.86 20.32) (xy 22.86 22.86)
 		)
@@
 					(unit 1)
 				)
+			)
+		)
+	)
+	(symbol
+		(lib_id "lcsc_imported:SMBJ60A TVS ")
+		(at 49.53 78.74 270)
+		(unit 1)
+		(exclude_from_sim no)
+		(in_bom yes)
+		(on_board yes)
+		(dnp no)
+		(property "Reference" "D1"
+			(at 52.07 78.1049 90)
+			(effects
+				(font
+					(size 1.27 1.27)
+				)
+				(justify left)
+			)
+		)
+		(property "Value" "TVS DIODE 60VWM 96.8VC SMB(DO-214AA)"
+			(at 46.482 69.596 0)
+			(effects
+				(font
+					(size 0.635 0.635)
+				)
+				(justify left)
+			)
+		)
+		(property "Footprint" "lcsc_footprints:C49066953_SMB_L4_5-W3_7-LS5_4-RD"
+			(at 39.37 78.74 0)
+			(effects
+				(font
+					(size 1.27 1.27)
+				)
+				(hide yes)
+			)
+		)
+		(property "Datasheet" "https://www.lcsc.com/datasheet/C49066953.pdf?spm=wm.sxq.inf.ggs___wm.fly.bg.7.xh&lcsc_vid=FANbVFRST1hfU1JfR1ZbXlBfEgcPVgcEQgNYBlVSEwAxVlNeQlBaXlFfQ1JYXjsOAxUeFF5JWBYZEEoKFBINSQcJGk4eFQsCAgIaSgADAwAHC0slRlRfVVBRWQkaCgg%3D"
+			(at 49.657 76.454 0)
+			(effects
+				(font
+					(size 1.27 1.27)
+				)
+				(hide yes)
+			)
+		)
+		(property "Description" "SMBJ60A TVS"
+			(at 49.53 78.74 0)
+			(effects
+				(font
+					(size 1.27 1.27)
+				)
+				(hide yes)
+			)
+		)
+		(property "LCSC" "C49066953"
+			(at 49.53 78.74 0)
+			(effects
+				(font
+					(size 1.27 1.27)
+				)
+				(hide yes)
+			)
+		)
+		(property "Manufacturer" "R+O(宏嘉诚)"
+			(at 49.53 78.74 0)
+			(effects
+				(font
+					(size 1.27 1.27)
+				)
+				(hide yes)
+			)
+		)
+		(pin "1"
+		)
+		(pin "2"
+		)
+		(instances
+			(project ""
+				(path "/daf77073-b189-4351-8636-4e7a5198e1b7/f3c2518b-d41d-4c2c-ab2c-6739c5137e70"
+					(reference "D1")
+					(unit 1)
+				)

Commit message: pdf of schematic added
Other:
- title: (none) -> LV Bridge
Changed lines of the file:
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@@
 	(generator_version "9.0")
 	(paper "A4")
+	(title_block
+		(title "LV Bridge")
+		(date "2026-07-27")
+		(rev "V0.1 for review")
+	)
 	(text "Gate driver pins"
 		(exclude_from_sim no)
